Commit message: Cleaned codebase, added scripts, Dockerized repo

File: ros2_ws/src/robot_slam/urdf/robot.urdf.xacro (robot description, xacro)
@@ -1,25 +1,35 @@
 <!-- urdf/robot.urdf.xacro -->
+<!-- Mount offsets are estimates — measure on the rover and update the <origin> values. -->
 <robot name="my_robot" xmlns:xacro="http://www.ros.org/wiki/xacro">
   <link name="base_link"/>
-  <!-- 2D LiDAR -->
+  <!-- Livox Mid-360 LiDAR. Child frame name must match the driver's frame_id
+       (livox_bringup lidar_frame, default livox_frame). -->
   <joint name="lidar_joint" type="fixed">
     <parent link="base_link"/>
-    <child link="laser"/>
+    <child link="livox_frame"/>
     <origin xyz="0.1 0.0 0.2" rpy="0 0 0"/>
   </joint>
-  <link name="laser"/>
-  <!-- OAK-D Lite -->
-  <joint name="camera_joint" type="fixed">
+  <link name="livox_frame"/>
+  <!-- OAK-D Pro body frame (REP-103: x forward, y left, z up) -->
+  <joint name="oakd_joint" type="fixed">
     <parent link="base_link"/>
-    <child link="camera_link"/>
+    <child link="oakd_link"/>
     <origin xyz="0.15 0.0 0.25" rpy="0 0 0"/>
   </joint>
-  <link name="camera_link"/>
-  <!-- IMU (Seeed XIAO) -->
-  <joint name="imu_joint" type="fixed">
-    <parent link="base_link"/>
-    <child link="base_imu_link"/>
-    <origin xyz="0.0 0.0 0.1" rpy="0 0 0"/>
+  <link name="oakd_link"/>
+  <!-- Optical frame (x right, y down, z forward) — frame_id of /oakd/color and /oakd/depth -->
+  <joint name="oakd_optical_joint" type="fixed">
+    <parent link="oakd_link"/>
+    <child link="oakd_camera_optical_frame"/>
+    <origin xyz="0 0 0" rpy="-1.5708 0 -1.5708"/>
   </joint>
-  <link name="base_imu_link"/>
+  <link name="oakd_camera_optical_frame"/>
+  <!-- OAK-D Pro onboard IMU. oakd_publisher rotates samples so this frame is
+       axis-aligned with oakd_link; keep rpy at zero. -->
+  <joint name="oakd_imu_joint" type="fixed">
+    <parent link="oakd_link"/>
+    <child link="oakd_imu_frame"/>
+    <origin xyz="0 0 0" rpy="0 0 0"/>
+  </joint>
+  <link name="oakd_imu_frame"/>
 </robot>
